File: spelaroo/spelaroo.kicad_pcb (KiCad board)
At the start: 2 copper layers, 93.8 x 87.3 mm, 19 parts, among them J1 USB_B_Micro, J2 Conn_01x14_Pin, J3 Micro_SD_Card, SW1 SW_Push, SW2 SW_Push, SW3 K1-1506DN-01, SW4 SW_Push, U1 ESP32-S3-WROOM-1, U2 LP2985-3.3, U3 OTJ-5

Commit message: addied things
Parts:
- added C3: 100nF, Capacitor_SMD:C_1206_3216Metric, B.Cu at (204.5, 61.9)
Routing:
- net +3.3V: track 105.8 -> 113.5 mm
- net GND: track 270.3 -> 277.9 mm

Commit message: fis
Parts:
- added C4: 10uF, Capacitor_SMD:C_1206_3216Metric, B.Cu at (238.1, 79.3)
- added C5: 100nF, Capacitor_SMD:C_1206_3216Metric, B.Cu at (234.2, 79.3)
- added C6: 10uF, Capacitor_SMD:C_1206_3216Metric, B.Cu at (215.1, 52.7)
- added C7: 10µF, Capacitor_SMD:C_1206_3216Metric, B.Cu at (224.9, 57.0)
- added C8: 10µF, Capacitor_SMD:C_1206_3216Metric, B.Cu at (186.0, 67.7)
- added C9: 100nF, Capacitor_SMD:C_1206_3216Metric, B.Cu at (185.9, 63.9)
- moved U1 47.5 mm to (220.3, 82.3)
- moved SW1 31.6 mm to (191.5, 79.8), turned to 90 degrees
- moved SW2 16.6 mm to (196.8, 79.7), turned to 90 degrees
- moved U3 3.26 mm to (204.8, 54.1)
- moved U2 2.97 mm to (225.2, 52.5)
- moved C3 2.32 mm to (206.0, 60.1)
- renumbered REF** to M1, REF** to M2, REF** to M3, REF** to M4
Connections:
- J3 pad 10: (no net) -> GND
Routing:
- net /RST_TFT: track 125.6 -> 22.2 mm, vias 3 -> 1
- net /CS_TFT: track 130.2 -> 33.0 mm, vias 3 -> 1
- net /DC: track 74.0 -> 24.5 mm, vias 6 -> 0
- net /LED: track 91.7 -> 43.2 mm, vias 5 -> 1
- net GND: track 277.9 -> 317.6 mm, vias 11 -> 1
- net /MOSI: track 102.8 -> 71.4 mm, vias 6 -> 2
- net /SCK: track 124.1 -> 95.9 mm, vias 7 -> 2
- net +3.3V: track 113.5 -> 139.3 mm, vias 6 -> 2
- net /boot: track 100.9 -> 75.8 mm
- net /MISO: track 109.3 -> 86.5 mm
- net /CS_SD: track 36.5 -> 58.7 mm, vias 4 -> 2
- net /d+: track 69.8 -> 51.7 mm, vias 4 -> 2
- net /3: track 35.3 -> 53.3 mm, vias 1 -> 0
- net /1: track 30.7 -> 46.9 mm
- net /2: track 33.3 -> 49.4 mm
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